File: hardware/segment-display-4x7-v2.kicad_pcb (KiCad board)
At the start: 2 copper layers, 65 x 25 mm, 32 parts, among them P1 CON-SENSOR2, P2 DEBUG, P3 BOOT, U1 XMC1XXX24, U2 TM1637, U3 SEGMENT_4X7, U4 DRILL, U5 DRILL, U6 DRILL, U7 DRILL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

Commit message: changed processor to XMC1100
Parts:
- U1: value XMC1XXX24 -> XMC1100
Changed lines of the file:
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@@
     (pad_drill 0.8)
     (pad_to_mask_clearance 0)
+    (solder_mask_min_width 0.25)
     (aux_axis_origin 176.9 165.9)
     (grid_origin 176.9 165.9)
@@
       (effects (font (size 0.3 0.3) (thickness 0.075)))
     )
-    (fp_text value XMC1XXX24 (at 0 0.8) (layer F.Fab)
-      (effects (font (size 0.3 0.3) (thickness 0.075)))
-    )
+    (fp_text value XMC1100 (at 0 0.8) (layer F.Fab)
+      (effects (font (size 0.3 0.3) (thickness 0.075)))
+    )
